File: SCART to VGA.kicad_pcb (KiCad board)
At the start: 2 copper layers, 44.4 x 63.5 mm, 14 parts, among them J1 SCART-F, J2 Conn_01x03_Male, J3 USB_B_Micro, J4 DB15_Female_HighDensity, J5 AudioJack3, U1 LM1881

Commit message: renamed gerber file
Parts:
- moved J4 6.93 mm to (103.6, 78.6)
