File: SCART to VGA.kicad_pcb (KiCad board)
At the start: 2 copper layers, 32.1 x 62.6 mm, 14 parts, among them J1 SCART-F, J2 Conn_01x03_Male, J3 USB_B_Micro, J4 DB15_Female_HighDensity, J5 AudioJack3, J6 V+ Select, U1 LM1881

Commit message: fixed routing for bypass cap
Fixed routing for LM1881 bypass cap so voltage input hits the cap first.
Routing:
- net Net-(C3-Pad1): track 18.6 -> 23.0 mm
Changed lines of the file:
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@@
     (visible_elements 7FFFFFFF)
     (pcbplotparams
-      (layerselection 0x010fc_ffffffff)
+      (layerselection 0x010f8_ffffffff)
       (usegerberextensions true)
       (usegerberattributes false)
@@
   (segment (start 100.6615 120.156) (end 100.6475 120.142) (width 0.25) (layer F.Cu) (net 4))
   (segment (start 100.6615 121.793) (end 100.6615 120.156) (width 0.25) (layer F.Cu) (net 4))
-  (segment (start 98.839 118.491) (end 98.331 118.999) (width 0.25) (layer F.Cu) (net 5))
-  (segment (start 100.6374 118.491) (end 98.839 118.491) (width 0.25) (layer F.Cu) (net 5))
   (segment (start 92.869 129.554) (end 94.234 128.189) (width 0.25) (layer F.Cu) (net 5))
   (segment (start 92.329 129.554) (end 92.869 129.554) (width 0.25) (layer F.Cu) (net 5))
   (segment (start 94.76 128.189) (end 96.139 129.568) (width 0.25) (layer F.Cu) (net 5))
   (segment (start 94.234 128.189) (end 94.76 128.189) (width 0.25) (layer F.Cu) (net 5))
-  (segment (start 97.856 118.999) (end 98.331 118.999) (width 0.25) (layer F.Cu) (net 5))
-  (segment (start 94.996 121.859) (end 97.856 118.999) (width 0.25) (layer F.Cu) (net 5))
-  (segment (start 94.234 128.189) (end 94.996 127.427) (width 0.25) (layer F.Cu) (net 5))
-  (segment (start 94.996 127.427) (end 94.996 121.859) (width 0.25) (layer F.Cu) (net 5))
+  (segment (start 98.839 118.491) (end 98.331 118.999) (width 0.25) (layer F.Cu) (net 5))
+  (segment (start 100.6374 118.491) (end 98.839 118.491) (width 0.25) (layer F.Cu) (net 5))
+  (segment (start 100.0024 117.856) (end 100.6374 118.491) (width 0.25) (layer F.Cu) (net 5))
+  (segment (start 96.647 117.856) (end 100.0024 117.856) (width 0.25) (layer F.Cu) (net 5))
+  (segment (start 94.234 128.189) (end 94.234 120.269) (width 0.25) (layer F.Cu) (net 5))
+  (segment (start 94.234 120.269) (end 96.647 117.856) (width 0.25) (layer F.Cu) (net 5))
   (segment (start 96.2025 96.8915) (end 96.2025 95.7415) (width 0.25) (layer F.Cu) (net 7))
   (segment (start 88.9 104.194) (end 96.2025 96.8915) (width 0.25) (layer F.Cu) (net 7))
