File: SCART to VGA.kicad_pcb (KiCad board)
At the start: 2 copper layers, 32.1 x 62.6 mm, 14 parts, among them J1 SCART-F, J2 Conn_01x03_Male, J3 USB_B_Micro, J4 DB15_Female_HighDensity, J5 AudioJack3, J6 V+ Select, U1 LM1881

Commit message: added jumper to make it easier to use without sync stripper
Parts:
- added JP1: SolderJumper-2_P1.3mm_Open_RoundedPad1.0x1.5mm, Jumper:SolderJumper-2_P1.3mm_Open_RoundedPad1.0x1.5mm, F.Cu at (93.5, 107.6)
Routing:
- net SYNC_OUT: track 67.2 -> 80.4 mm, vias 0 -> 1
- net SYNC_IN: track 46.9 -> 56.0 mm, vias 1 -> 2
Other:
- board text added: "Close for use w/o stripper"
Changed lines of the file:
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@@
   (general
     (thickness 1.6)
-    (drawings 9)
-    (tracks 116)
+    (drawings 14)
+    (tracks 127)
     (zones 0)
-    (modules 14)
+    (modules 15)
     (nets 33)
   )
@@
     (mod_text_size 1 1)
     (mod_text_width 0.15)
-    (pad_size 1.8 2.5)
-    (pad_drill 0.8)
+    (pad_size 1 0.5)
+    (pad_drill 0)
     (pad_to_mask_clearance 0.051)
     (solder_mask_min_width 0.25)
@@
     (add_net SYNC_OUT)
   )
+  (module Jumper:SolderJumper-2_P1.3mm_Open_RoundedPad1.0x1.5mm (layer F.Cu)
+    (at 93.5 107.6 90)
+    (descr "SMD Solder Jumper, 1x1.5mm, rounded Pads, 0.3mm gap, open")
+    (tags "solder jumper open")
+    (attr virtual)
+    (fp_text reference JP1 (at 0.1 -1.95 90) (layer F.SilkS)
+      (effects (font (size 1 1) (thickness 0.15)))
+    )
+    (fp_text value SolderJumper-2_P1.3mm_Open_RoundedPad1.0x1.5mm (at 0 1.9 90) (layer F.Fab)
+      (effects (font (size 1 1) (thickness 0.15)))
+    )
+    (fp_line (start 1.65 1.25) (end -1.65 1.25) (layer F.CrtYd) (width 0.05))
+    (fp_line (start 1.65 1.25) (end 1.65 -1.25) (layer F.CrtYd) (width 0.05))
+    (fp_line (start -1.65 -1.25) (end -1.65 1.25) (layer F.CrtYd) (width 0.05))
+    (fp_line (start -1.65 -1.25) (end 1.65 -1.25) (layer F.CrtYd) (width 0.05))
+    (fp_line (start -0.7 -1) (end 0.7 -1) (layer F.SilkS) (width 0.12))
+    (fp_line (start 1.4 -0.3) (end 1.4 0.3) (layer F.SilkS) (width 0.12))
+    (fp_line (start 0.7 1) (end -0.7 1) (layer F.SilkS) (width 0.12))
+    (fp_line (start -1.4 0.3) (end -1.4 -0.3) (layer F.SilkS) (width 0.12))
+    (fp_arc (start -0.7 -0.3) (end -0.7 -1) (angle -90) (layer F.SilkS) (width 0.12))
+    (fp_arc (start -0.7 0.3) (end -1.4 0.3) (angle -90) (layer F.SilkS) (width 0.12))
+    (fp_arc (start 0.7 0.3) (end 0.7 1) (angle -90) (layer F.SilkS) (width 0.12))
+    (fp_arc (start 0.7 -0.3) (end 1.4 -0.3) (angle -90) (layer F.SilkS) (width 0.12))
+    (pad 2 smd custom (at 0.65 0 90) (size 1 0.5) (layers F.Cu F.Mask)
+      (net 2 SYNC_IN) (zone_connect 2)
+      (options (clearance outline) (anchor rect))
+      (primitives
+        (gr_circle (center 0 0.25) (end 0.5 0.25) (width 0))
+        (gr_circle (center 0 -0.25) (end 0.5 -0.25) (width 0))
+        (gr_poly (pts
+           (xy 0 -0.75) (xy -0.5 -0.75) (xy -0.5 0.75) (xy 0 0.75)) (width 0))
+      ))
+    (pad 1 smd custom (at -0.65 0 90) (size 1 0.5) (layers F.Cu F.Mask)
+      (net 19 SYNC_OUT) (zone_connect 2)
+      (options (clearance outline) (anchor rect))
+      (primitives
+        (gr_circle (center 0 0.25) (end 0.5 0.25) (width 0))
+        (gr_circle (center 0 -0.25) (end 0.5 -0.25) (width 0))
+        (gr_poly (pts
+           (xy 0 -0.75) (xy 0.5 -0.75) (xy 0.5 0.75) (xy 0 0.75)) (width 0))
+      ))
+  )
   (module Tinkerplunk:CUI_SJ1-3533NG (layer F.Cu)
     (at 100.15 98.1 90)
@@
       (effects (font (size 1.6891 1.6891) (thickness 0.1778)) (justify left bottom))
     )
-    (fp_text user 1 (at 19.939 2.286 270) (layer F.SilkS)
+    (fp_text user 1 (at 19.629 5.3595 270) (layer F.SilkS)
       (effects (font (size 1.2065 1.2065) (thickness 0.127)) (justify left bottom))
     )
-    (fp_text user 21 (at -21.336 2.286 270) (layer F.SilkS)
+    (fp_text user 21 (at -21.336 4.3595 270) (layer F.SilkS)
       (effects (font (size 1.2065 1.2065) (thickness 0.127)) (justify left bottom))
     )
@@
     )
   )
+  (gr_line (start 93 105) (end 93.5 105.5) (layer F.SilkS) (width 0.12))
+  (gr_line (start 94 105) (end 93 105) (layer F.SilkS) (width 0.12))
+  (gr_line (start 93.5 105.5) (end 94 105) (layer F.SilkS) (width 0.12))
+  (gr_line (start 93.5 104) (end 93.5 105.5) (layer F.SilkS) (width 0.12))
+  (gr_text "Close for use\nw/o stripper" (at 92.9 98.65 90) (layer F.SilkS)
+    (effects (font (size 1 1) (thickness 0.25)))
+  )
   (gr_line (start 105.8545 74.93) (end 105.8545 137.541) (layer Edge.Cuts) (width 0.05))
   (gr_line (start 73.787 137.541) (end 105.8545 137.541) (layer Edge.Cuts) (width 0.05))
@@
   (segment (start 101.6 124.2428) (end 101.6 124.333012) (width 0.25) (layer F.Cu) (net 2))
   (segment (start 101.6 124.898697) (end 101.6 124.333012) (width 0.25) (layer B.Cu) (net 2))
+  (via (at 95.5 107) (size 0.8) (drill 0.4) (layers F.Cu B.Cu) (net 2))
+  (segment (start 93.5 106.95) (end 95.45 106.95) (width 0.25) (layer F.Cu) (net 2))
+  (segment (start 95.45 106.95) (end 95.5 107) (width 0.25) (layer F.Cu) (net 2))
+  (segment (start 97.9165 109.4165) (end 101.6 109.4165) (width 0.25) (layer B.Cu) (net 2))
+  (segment (start 95.5 107) (end 97.9165 109.4165) (width 0.25) (layer B.Cu) (net 2))
   (segment (start 92.477 136.048) (end 98.877 136.048) (width 0.25) (layer F.Cu) (net 3))
   (segment (start 92.877 135.648) (end 92.477 136.048) (width 0.25) (layer F.Cu) (net 3))
@@
   (segment (start 102.7 99.906) (end 103.632 100.838) (width 0.25) (layer B.Cu) (net 19))
   (segment (start 103.632 100.838) (end 103.632 128.983) (width 0.25) (layer B.Cu) (net 19))
+  (via (at 100 104.499992) (size 0.8) (drill 0.4) (layers F.Cu B.Cu) (net 19))
+  (segment (start 93.5 108.25) (end 96.249992 108.25) (width 0.25) (layer F.Cu) (net 19))
+  (segment (start 99.600001 104.899991) (end 100 104.499992) (width 0.25) (layer F.Cu) (net 19))
+  (segment (start 96.249992 108.25) (end 99.600001 104.899991) (width 0.25) (layer F.Cu) (net 19))
+  (segment (start 103.632 100.867992) (end 103.632 100.838) (width 0.25) (layer B.Cu) (net 19))
+  (segment (start 100 104.499992) (end 103.632 100.867992) (width 0.25) (layer B.Cu) (net 19))
   (segment (start 92.569 131.304) (end 92.329 131.304) (width 0.25) (layer F.Cu) (net 32))
   (segment (start 94.077 133.348) (end 94.077 132.812) (width 0.25) (layer F.Cu) (net 32))
