File: SCART to VGA.sch (KiCad schematic (older format))
At the start: 13 parts, among them J1 SCART-F, J2 Conn_01x03_Male, J3 USB_B_Micro, J4 DB15_Female_HighDensity, J5 AudioJack3, U1 LM1881

Commit message: Created branch
Branch where the SCART head lays on top of the PCB for direct plug in with a male hd-15 port.
Parts:
- C3: footprint Capacitor_SMD:CP_Elec_5x5.3 -> Capacitor_Tantalum_SMD:CP_EIA-3216-18_Kemet-A_Pad1.58x1.35mm_HandSolder
- J4: footprint Connector_Dsub:DSUB-15-HD_Female_Horizontal_P2.29x1.98mm_EdgePinOffset3.03mm_Housed_MountingHolesOffset4.94mm -> Connector_Dsub:DSUB-15-HD_Male_Horizontal_P2.29x1.98mm_EdgePinOffset3.03mm_Housed_MountingHolesOffset4.94mm
- J5: footprint digikey-footprints:Headphone_Jack_3.5mm_SJ1-3523N -> SJ-3523-SMT-TR:CUI_SJ-3523-SMT-TR
Changed lines of the file:
@@
 EESchema Schematic File Version 4
+LIBS:SCART to VGA-cache
 EELAYER 29 0
 EELAYER END
@@
 F 0 "J4" H 7100 4617 50  0000 C CNN
 F 1 "DB15_Female_HighDensity" H 7100 4526 50  0000 C CNN
-F 2 "Connector_Dsub:DSUB-15-HD_Female_Horizontal_P2.29x1.98mm_EdgePinOffset3.03mm_Housed_MountingHolesOffset4.94mm" H 6150 4150 50  0001 C CNN
+F 2 "Connector_Dsub:DSUB-15-HD_Male_Horizontal_P2.29x1.98mm_EdgePinOffset3.03mm_Housed_MountingHolesOffset4.94mm" H 6150 4150 50  0001 C CNN
 F 3 " ~" H 6150 4150 50  0001 C CNN
 	1    7100 3750
@@
 F 0 "J5" H 6820 4783 50  0000 R CNN
 F 1 "AudioJack3" H 6820 4874 50  0000 R CNN
-F 2 "digikey-footprints:Headphone_Jack_3.5mm_SJ1-3523N" H 7100 4850 50  0001 C CNN
+F 2 "SJ-3523-SMT-TR:CUI_SJ-3523-SMT-TR" H 7100 4850 50  0001 C CNN
 F 3 "~" H 7100 4850 50  0001 C CNN
 	1    7100 4850
@@
 F 0 "C3" H 6262 1704 50  0000 R CNN
 F 1 "10uF" H 6262 1795 50  0000 R CNN
-F 2 "Capacitor_SMD:CP_Elec_5x5.3" H 6350 1750 50  0001 C CNN
+F 2 "Capacitor_Tantalum_SMD:CP_EIA-3216-18_Kemet-A_Pad1.58x1.35mm_HandSolder" H 6350 1750 50  0001 C CNN
 F 3 "~" H 6350 1750 50  0001 C CNN
 	1    6350 1750

Commit message: 1.1 Update
Moved things around, made cutout for headphone jack, changed headphone jack part, added jumper for getting voltage optionally from the SCART socket.
Parts:
- added J6: Voltage Select, Connector_PinHeader_2.54mm:PinHeader_1x02_P2.54mm_Vertical, symbol Connector:Conn_01x02_Male
- J5: footprint SJ-3523-SMT-TR:CUI_SJ-3523-SMT-TR -> SJ1-3533NG:CUI_SJ1-3533NG
Connections:
- net at J1.8 (P8): now also J6.1 (Pin_1)
- net SCART_VOLTAGE: now reaches FB1.1, J3.1 (VBUS)
- net SCART_VOLTAGE: now also J6.2 (Pin_2)
- no-connect marks 16 -> 15
Changed lines of the file:
@@
 F 0 "J5" H 6820 4783 50  0000 R CNN
 F 1 "AudioJack3" H 6820 4874 50  0000 R CNN
-F 2 "SJ-3523-SMT-TR:CUI_SJ-3523-SMT-TR" H 7100 4850 50  0001 C CNN
+F 2 "SJ1-3533NG:CUI_SJ1-3533NG" H 7100 4850 50  0001 C CNN
 F 3 "~" H 7100 4850 50  0001 C CNN
 	1    7100 4850
@@
 NoConn ~ 2050 4700
 NoConn ~ 2050 4900
-NoConn ~ 3250 4200
 NoConn ~ 3250 4000
 NoConn ~ 3250 3800
@@
 Text GLabel 6400 3650 0    50   Input ~ 0
 GND
+$Comp
+L Connector:Conn_01x02_Male J6
+U 1 1 5CC4DF98
+P 3950 4400
+F 0 "J6" V 4104 4212 50  0000 R CNN
+F 1 "Voltage Select" V 4013 4212 50  0000 R CNN
+F 2 "Connector_PinHeader_2.54mm:PinHeader_1x02_P2.54mm_Vertical" H 3950 4400 50  0001 C CNN
+F 3 "~" H 3950 4400 50  0001 C CNN
+	1    3950 4400
+	0    -1   -1   0
+$EndComp
+Wire Wire Line
+	3250 4200 3950 4200
+Wire Wire Line
+	4050 4200 4750 4200
+Text GLabel 4750 4200 2    50   Input ~ 0
+SCART_VOLTAGE
+Text GLabel 6850 1300 2    50   Input ~ 0
+SCART_VOLTAGE
+Wire Wire Line
+	6850 1300 6200 1300
+Connection ~ 6200 1300
 $EndSCHEMATC

Commit message: saving
Parts:
- U1: symbol SCART_to_DVI-A_Compact-eagle-import:LM1881 -> SCART-to-VGA-rescue:LM1881-SCART_to_DVI-A_Compact-eagle-import
Changed lines of the file:
@@
 $EndComp
 $Comp
-L SCART_to_DVI-A_Compact-eagle-import:LM1881 U1
+L SCART-to-VGA-rescue:LM1881-SCART_to_DVI-A_Compact-eagle-import U1
 U 1 1 5CBCF61B
 P 5300 2150
